Commit message: Add files via upload

File: Singlearm_Sim/Singlearm/singlearm_description/urdf/link_to_joint.xacro (robot description, xacro)
@@ -33,5 +33,5 @@
   </xacro:macro>
   <xacro:macro name="m_link_cylinder"
-               params="name origin_xyz origin_rpy mass ixx ixy ixz iyy iyz izz mesh_file mesh_scale">
+               params="name origin_xyz origin_rpy vis_rpy vis_xyz mass ixx ixy ixz iyy iyz izz mesh_file mesh_scale">
     <link name="${name}">
       <inertial>
@@ -60,6 +60,6 @@
       <visual>
         <origin
-                rpy="${origin_rpy}"
-                xyz="${origin_xyz}" />
+                rpy="${vis_rpy}"
+                xyz="${vis_xyz}" />
         <geometry>
           <mesh

File: Singlearm_Sim/Singlearm/singlearm_description/urdf/robot_parameter.xacro (robot description, xacro)
@@ -20,10 +20,10 @@
   <xacro:property name="L6_mass" value="0.0612"/>
 <!-- link_inertia -->
-  <xacro:property name="base_link_ixx" value="0.0"/>
-  <xacro:property name="base_link_ixy" value="0.0"/>
-  <xacro:property name="base_link_ixz" value="0.0"/>
-  <xacro:property name="base_link_iyy" value="0.0"/>
-  <xacro:property name="base_link_izz" value="0.0"/>
-  <xacro:property name="base_link_iyz" value="0.0"/>
+  <xacro:property name="base_link_ixx" value="0"/>
+  <xacro:property name="base_link_ixy" value="0"/>
+  <xacro:property name="base_link_ixz" value="0"/>
+  <xacro:property name="base_link_iyy" value="0"/>
+  <xacro:property name="base_link_izz" value="0"/>
+  <xacro:property name="base_link_iyz" value="0"/>
   <xacro:property name="L1_ixx" value="0.096344"/>
   <xacro:property name="L1_ixy" value="0.0000230"/>

File: Singlearm_Sim/Singlearm/singlearm_description/urdf/singlearm.xacro (robot description, xacro)
@@ -26,4 +26,6 @@
 			iyz="${base_link_iyz}"
 			izz="${base_link_izz}"
+			vis_rpy="0 0 0"
+			vis_xyz="0 0 0"
 			mesh_file="package://singlearm_description/meshes/base_link.STL"
 			mesh_scale="0.001 0.001 0.001"
@@ -47,5 +49,5 @@
 			mass="${L1_mass}"
 			origin_rpy="0 0 0"
-			origin_xyz="0 0 0"
+			origin_xyz="0.0671349 -0.0000384 0.0588309"
 			ixx="${L1_ixx}"
 			ixy="${L1_ixy}"
@@ -54,4 +56,6 @@
 			iyz="${L1_iyz}"
 			izz="${L1_izz}"
+			vis_rpy="0 0 0"
+			vis_xyz="0 0 0"
 			mesh_file="package://singlearm_description/meshes/L1.STL"
 			mesh_scale="0.001 0.001 0.001"
@@ -74,5 +78,5 @@
 			mass="${L2_mass}"
 			origin_rpy="0 0 0"
-			origin_xyz="0 0 0"
+			origin_xyz="0.0724494 0.0167624 0.0001735"
 			ixx="${L2_ixx}"
 			ixy="${L2_ixy}"
@@ -81,4 +85,6 @@
 			iyz="${L2_iyz}"
 			izz="${L2_izz}"
+			vis_rpy="0 0 0"
+			vis_xyz="0 0 0"
 			mesh_file="package://singlearm_description/meshes/L2.STL"
 			mesh_scale="0.001 0.001 0.001"
@@ -101,5 +107,5 @@
 			mass="${L3_mass}"
 			origin_rpy="0 0 0"
-			origin_xyz="0 0 0"
+			origin_xyz="0.0001081 0.0015321 -0.1744158"
 			ixx="${L3_ixx}"
 			ixy="${L3_ixy}"
@@ -108,4 +114,6 @@
 			iyz="${L3_iyz}"
 			izz="${L3_izz}"
+			vis_rpy="0 0 0"
+			vis_xyz="0 0 0"
 			mesh_file="package://singlearm_description/meshes/L3.STL"
 			mesh_scale="0.001 0.001 0.001"
@@ -128,5 +136,5 @@
 			mass="${L4_mass}"
 			origin_rpy="0 0 0"
-			origin_xyz="0 0 0"
+			origin_xyz="-0.0230881 -0.0145184 -0.129937"
 			ixx="${L4_ixx}"
 			ixy="${L4_ixy}"
@@ -135,4 +143,6 @@
 			iyz="${L4_iyz}"
 			izz="${L4_izz}"
+			vis_rpy="0 0 0"
+			vis_xyz="0 0 0"
 			mesh_file="package://singlearm_description/meshes/L4.STL"
 			mesh_scale="0.001 0.001 0.001"
@@ -155,5 +165,5 @@
 			mass="${L5_mass}"
 			origin_rpy="0 0 0"
-			origin_xyz="0 0 0"
+			origin_xyz="0.0192632 -0.0014654 -0.1592943"
 			ixx="${L5_ixx}"
 			ixy="${L5_ixy}"
@@ -162,4 +172,6 @@
 			iyz="${L5_iyz}"
 			izz="${L5_izz}"
+			vis_rpy="0 0 0"
+			vis_xyz="0 0 0"
 			mesh_file="package://singlearm_description/meshes/L5.STL"
 			mesh_scale="0.001 0.001 0.001"
@@ -182,5 +194,5 @@
 			mass="${L6_mass}"
 			origin_rpy="0 0 0"
-			origin_xyz="0 0 0"
+			origin_xyz="0 0 -0.0066153"
 			ixx="${L6_ixx}"
 			ixy="${L6_ixy}"
@@ -189,4 +201,6 @@
 			iyz="${L6_iyz}"
 			izz="${L6_izz}"
+			vis_rpy="0 0 0"
+			vis_xyz="0 0 0"
 			mesh_file="package://singlearm_description/meshes/L6.STL"
 			mesh_scale="0.001 0.001 0.001"
