Commit message: Prepare the AppSci
finished

File: Singlearm_Sim/Singlearm/singlearm_description/urdf/elfin3_experiment1.urdf.xacro (robot description, xacro)
@@ -394,5 +394,5 @@
     <origin
       xyz="0 -0.1065 0"
-      rpy="${-PI} 0 ${-PI}" />
+      rpy="${PI} 0 ${PI}" />
     <parent
       link="elfin_link5" />
@@ -455,6 +455,14 @@
     <inertial>
       <mass value="0.01" />
-      <origin xyz="0 0 0" rpy="0 0 0"/>
-      <inertia ixx="0.01" ixy="0" ixz="0" iyy="0.01" iyz="0" izz="0.01" />
+      <origin
+              xyz="0 0 0"
+              rpy="0 0 0"/>
+      <inertia
+              ixx="0.01"
+              ixy="0"
+              ixz="0"
+              iyy="0.01"
+              iyz="0"
+              izz="0.01" />
     </inertial>
   </link>
@@ -462,5 +470,7 @@
     <parent link="elfin_ft_sensor_link"/>
     <child link="elfin_tool"/>
-    <origin xyz="0 -0.05 0" rpy="0 0 0" />
+    <origin
+            xyz="0 -0.05 0"
+            rpy="0 0 0" />
   </joint>
   <link name="elfin_tool_ball">
@@ -472,5 +482,7 @@
     </collision>
     <visual>
-      <origin xyz="0 0 0" rpy="0 0 0" />
+      <origin
+              xyz="0 0 0"
+              rpy="0 0 0" />
       <geometry>
         <sphere radius="0.02"/>
@@ -479,6 +491,14 @@
     <inertial>
       <mass value="0.01" />
-      <origin xyz="0 0 0" rpy="0 0 0"/>
-      <inertia ixx="0.01" ixy="0" ixz="0" iyy="0.01" iyz="0" izz="0.01" />
+      <origin
+              xyz="0 0 0"
+              rpy="0 0 0"/>
+      <inertia
+              ixx="0.01"
+              ixy="0"
+              ixz="0"
+              iyy="0.01"
+              iyz="0"
+              izz="0.01" />
     </inertial>
   </link>
@@ -486,5 +506,7 @@
     <parent link="elfin_tool"/>
     <child link="elfin_tool_ball"/>
-    <origin xyz="0 -0.04 0" rpy="0 0 0" />
+    <origin
+            xyz="0 -0.04 0"
+            rpy="0 0 0" />
   </joint>
 </robot>

Commit message: Gazebo with rviz & rqt
rqt added

File: Singlearm_Sim/Singlearm/singlearm_description/urdf/elfin3_experiment1.urdf.xacro (robot description, xacro)
@@ -490,5 +490,5 @@
     </visual>
     <inertial>
-      <mass value="0.01" />
+      <mass value="5.0" />
       <origin
               xyz="0 0 0"
